Commit message: create servo controller

File: urdf/burt.urdf (robot description, URDF)
Before this commit: robot pi_robot, 5 links, 4 joints
Links:
- removed link arm_2
- removed link arm_2_1
Joints:
- removed joint arm_2_to_arm_2_1
- removed joint base_to_arm_2
- joint arm_1_to_arm_1_1: limit lower=-1.57079632679 upper=3.14159265359 effort=1000.0 velocity=10 -> lower=-3.14159 upper=3.14159 effort=1000.0 velocity=10
- joint base_to_arm_1: limit lower=-1.57079632679 upper=3.14159265359 effort=1000.0 velocity=10 -> lower=-3.14159 upper=3.14159 effort=1000.0 velocity=10

Commit message: implement simulation

File: urdf/burt.urdf (robot description, URDF)
Before this commit: robot pi_robot, 3 links, 2 joints
Links:
- removed link arm_1
- removed link arm_1_1
- added link bl_foot, mass 0.01; collision sphere radius=0.026; visual sphere radius=0.026
- added link bl_hip_link, mass 0.1; visual box size=0.04 0.03 0.04
- added link bl_lower_link, mass 0.05; visual box size=0.025 0.025 0.074
- added link bl_upper_link, mass 0.1; visual box size=0.03 0.03 0.10
- added link br_foot, mass 0.01; collision sphere radius=0.026; visual sphere radius=0.026
- added link br_hip_link, mass 0.1; visual box size=0.04 0.03 0.04
- added link br_lower_link, mass 0.05; visual box size=0.025 0.025 0.074
- added link br_upper_link, mass 0.1; visual box size=0.03 0.03 0.10
- added link fl_foot, mass 0.01; collision sphere radius=0.026; visual sphere radius=0.026
- added link fl_hip_link, mass 0.1; visual box size=0.04 0.03 0.04
- added link fl_lower_link, mass 0.05; visual box size=0.025 0.025 0.074
- added link fl_upper_link, mass 0.1; visual box size=0.03 0.03 0.10
- added link fr_foot, mass 0.01; collision sphere radius=0.026; visual sphere radius=0.026
- added link fr_hip_link, mass 0.1; visual box size=0.04 0.03 0.04
- added link fr_lower_link, mass 0.05; visual box size=0.025 0.025 0.074
- added link fr_upper_link, mass 0.1; visual box size=0.03 0.03 0.10
- link base_link: mass .0 -> 1.0; geometry collision box size=0.18 0.12 0.05; visual box size=0.18 0.12 0.05
Joints:
- removed joint arm_1_to_arm_1_1
- removed joint base_to_arm_1
- added joint bl_abduction: type revolute, parent base_link, child bl_hip_link, origin xyz=-0.09 0.06 0 rpy=0 0 0, axis 1 0 0, limit lower=-1.5708 upper=1.5708 effort=1000.0 velocity=10
- added joint bl_foot_joint: type fixed, parent bl_lower_link, child bl_foot, origin xyz=0 0 -0.074 rpy=0 0 0
- added joint bl_hip: type revolute, parent bl_hip_link, child bl_upper_link, origin xyz=0 0.03 0 rpy=0 0 0, axis 0 1 0, limit lower=-3.14159 upper=3.14159 effort=1000.0 velocity=10
- added joint bl_knee: type revolute, parent bl_upper_link, child bl_lower_link, origin xyz=0 0 -0.10 rpy=0 0 0, axis 0 1 0, limit lower=-3.14159 upper=3.14159 effort=1000.0 velocity=10
- added joint br_abduction: type revolute, parent base_link, child br_hip_link, origin xyz=-0.09 -0.06 0 rpy=0 0 0, axis 1 0 0, limit lower=-1.5708 upper=1.5708 effort=1000.0 velocity=10
- added joint br_foot_joint: type fixed, parent br_lower_link, child br_foot, origin xyz=0 0 -0.074 rpy=0 0 0
- added joint br_hip: type revolute, parent br_hip_link, child br_upper_link, origin xyz=0 -0.03 0 rpy=0 0 0, axis 0 1 0, limit lower=-3.14159 upper=3.14159 effort=1000.0 velocity=10
- added joint br_knee: type revolute, parent br_upper_link, child br_lower_link, origin xyz=0 0 -0.10 rpy=0 0 0, axis 0 1 0, limit lower=-3.14159 upper=3.14159 effort=1000.0 velocity=10
- added joint fl_abduction: type revolute, parent base_link, child fl_hip_link, origin xyz=0.09 0.06 0 rpy=0 0 0, axis 1 0 0, limit lower=-1.5708 upper=1.5708 effort=1000.0 velocity=10
- added joint fl_foot_joint: type fixed, parent fl_lower_link, child fl_foot, origin xyz=0 0 -0.074 rpy=0 0 0
- added joint fl_hip: type revolute, parent fl_hip_link, child fl_upper_link, origin xyz=0 0.03 0 rpy=0 0 0, axis 0 1 0, limit lower=-3.14159 upper=3.14159 effort=1000.0 velocity=10
- added joint fl_knee: type revolute, parent fl_upper_link, child fl_lower_link, origin xyz=0 0 -0.10 rpy=0 0 0, axis 0 1 0, limit lower=-3.14159 upper=3.14159 effort=1000.0 velocity=10
- added joint fr_abduction: type revolute, parent base_link, child fr_hip_link, origin xyz=0.09 -0.06 0 rpy=0 0 0, axis 1 0 0, limit lower=-1.5708 upper=1.5708 effort=1000.0 velocity=10
- added joint fr_foot_joint: type fixed, parent fr_lower_link, child fr_foot, origin xyz=0 0 -0.074 rpy=0 0 0
- added joint fr_hip: type revolute, parent fr_hip_link, child fr_upper_link, origin xyz=0 -0.03 0 rpy=0 0 0, axis 0 1 0, limit lower=-3.14159 upper=3.14159 effort=1000.0 velocity=10
- added joint fr_knee: type revolute, parent fr_upper_link, child fr_lower_link, origin xyz=0 0 -0.10 rpy=0 0 0, axis 0 1 0, limit lower=-3.14159 upper=3.14159 effort=1000.0 velocity=10
